File: hardware/Hermes/Hermes.kicad_pcb (KiCad board)
At the start: 2 copper layers, 78.6 x 61.9 mm, 5 parts, among them SW1 SW_Push, U1 HC-SR04

Commit message: Update Readme with wiring diagram and project purpose; adjust PCB design dimensions
Other:
- board size 78.6 x 61.9 mm -> 78.6 x 59.4 mm
Changed lines of the file:
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@@
 	(gr_rect
 		(start 138.1125 66.675)
-		(end 216.69375 128.5875)
+		(end 216.69375 126.0475)
 		(stroke
 			(width 0.05)
